File: VCU_v1/can3.kicad_sch (KiCad schematic)
At the start: 4 parts, among them U13 MCP2562 E/SN

Commit message: p dih r
Parts:
- added R28, R29, R30, R90: 0, Resistor_SMD:R_0805_2012Metric_Pad1.20x1.40mm_HandSolder, symbol bfr_resistors:RMCF0805ZT0R00
Connections:
- net +3.3V: now also R29.2; no longer C28.1, U13.5 (VIO)
- net +5V: now also R30.2; no longer U13. (VSS)
- net CAN3_L: no longer JP4.1 (A)
- net RX: now also R28.1; no longer U13.4 (RXD)
- net TX: now also R90.1; no longer U13.1 (TXD)
- new net: R28.2, U13.4 (RXD)
- new net: R30.1, U13. (VSS)
- new net: R90.2, U13.1 (TXD)
- new net: C28.1, R29.1, U13.5 (VIO)

Commit message: v1 schematic (actually) complete, let the layout commence
Parts:
- removed C28: 100n, Capacitor_SMD:C_0603_1608Metric_Pad1.08x0.95mm_HandSolder, symbol BFR Capacitors:06035C104KAT2A
- removed JP4: Jumper_3_Open, symbol Jumper:Jumper_3_Open
- removed R21: 120, Resistor_SMD:R_0603_1608Metric_Pad0.98x0.95mm_HandSolder, symbol BFR Resistors:RMCF0603FT120R
- removed R28, R29, R30, R90: 0, Resistor_SMD:R_0805_2012Metric_Pad1.20x1.40mm_HandSolder, symbol bfr_resistors:RMCF0805ZT0R00
- removed U13: MCP2562 E/SN, symbol MCP2562-CAN_Transceiver:MCP2562-E/SN
Other:
- note removed: "use jumper to terminate/unterminate CAN"
