File: VCU_v1/Bucks.kicad_sch (KiCad schematic)
At the start: 31 parts, among them U1 TPS5430, U2 TPS5430

Commit message: begin pcb design
Parts:
- L1: footprint SMTU2032-C:Untitled -> SER2211-333MED:Untitled
Changed lines of the file:
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@@
 			)
 		)
-		(property "Footprint" "SMTU2032-C:Untitled"
+		(property "Footprint" "SER2211-333MED:Untitled"
 			(at 173.99 114.3 0)
 			(effects

Commit message: omids wisdom came all over my power converters
Parts:
- C12: Digikey P/N (none) -> P12395-ND; Mouser P/N 667-EEU-FM1V151B -> 667-EEU-FM1H151B
Changed lines of the file:
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@@
 			)
 		)
-		(property "Description" "EEU-FM1V151B"
+		(property "Description" "EEU-FM1V151B 50V 150uF electrolytic capacitor"
 			(at 205.74 118.11 0)
 			(effects
@@
 			)
 		)
-		(property "Digikey P/N" ""
+		(property "Digikey P/N" "P12395-ND "
 			(at 205.994 130.302 0)
 			(effects
@@
 			)
 		)
-		(property "Mouser P/N" "667-EEU-FM1V151B "
+		(property "Mouser P/N" "667-EEU-FM1H151B "
 			(at 205.74 134.112 0)
 			(effects

Commit message: vcu placements complete
Parts:
- D3, D4: footprint LED_SMD:LED_0201_0603Metric_Pad0.64x0.40mm_HandSolder -> LED_SMD:LED_0603_1608Metric_Pad1.05x0.95mm_HandSolder
Changed lines of the file:
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@@
 			)
 		)
-		(property "Footprint" "LED_SMD:LED_0201_0603Metric_Pad0.64x0.40mm_HandSolder"
+		(property "Footprint" "LED_SMD:LED_0603_1608Metric_Pad1.05x0.95mm_HandSolder"
 			(at 220.98 125.73 0)
 			(effects
@@
 			)
 		)
-		(property "Footprint" "LED_SMD:LED_0201_0603Metric_Pad0.64x0.40mm_HandSolder"
+		(property "Footprint" "LED_SMD:LED_0603_1608Metric_Pad1.05x0.95mm_HandSolder"
 			(at 222.25 59.69 0)
 			(effects

Commit message: almost done i promise
Parts:
- removed C1: 100u, Capacitor_THT:CP_Radial_D8.0mm_P3.50mm, symbol BFR Capacitors:50ZLH100MEFC8X11.5
- removed C12: 150u, Capacitor_THT:CP_Radial_D8.0mm_P3.50mm, symbol BFR Capacitors:50ZLH100MEFC8X11.5
- removed C3, C5: 10u, Capacitor_SMD:C_0603_1608Metric_Pad1.08x0.95mm_HandSolder, symbol BFR Capacitors:CL10A106KP8NNNC
- removed C7: 10n, Capacitor_SMD:C_0603_1608Metric_Pad1.08x0.95mm_HandSolder, symbol BFR Capacitors:VJ0603Y103KXAAC
- removed C9: 220p, Capacitor_SMD:C_0603_1608Metric_Pad1.08x0.95mm_HandSolder, symbol BFR Capacitors:06035C221J4Z2A
- removed D1: B340LA-13-F, Diode_SMD:D_SMA_Handsoldering, symbol .Diode-Schottky:B340LA-13-F
- removed D3: GREEN LED, LED_SMD:LED_0603_1608Metric_Pad1.05x0.95mm_HandSolder, symbol Device:LED
- removed L1: 33u, SER2211-333MED:Untitled, symbol Device:L
- removed R1: 56, Resistor_SMD:R_0603_1608Metric_Pad0.98x0.95mm_HandSolder, symbol BFR Resistors:RMCF0603FT56R0
- removed R3: 10k, Resistor_SMD:R_0603_1608Metric_Pad0.98x0.95mm_HandSolder, symbol BFR Resistors:RMCF0603FT10K0
- removed R4: 620, Resistor_SMD:R_0603_1608Metric_Pad0.98x0.95mm_HandSolder, symbol BFR Resistors:RMCF0603FT620R
- removed R7, R8: 220, Resistor_SMD:R_0603_1608Metric_Pad0.98x0.95mm_HandSolder, symbol BFR Resistors:RMCF0603FT220R
- removed TP2: RH-5015, TestPoint:TestPoint_Keystone_5015_Micro_Mini, symbol .Test-Point:RH-5015
- removed U1: TPS5430, TPS5430DDAR:Untitled, symbol TPS5430:TPS5430
- added R1: 1.0k, Resistor_SMD:R_0603_1608Metric_Pad0.98x0.95mm_HandSolder, symbol BFR Resistors:RMCF0603FT1K00
Connections:
- net 5V-out: now also R1.2
- net at D4.2 (A): now also R1.1
- no-connect marks 6 -> 3
Other:
- note removed: "24V-20V Buck"
