File: VCU_v1/VCU_v1.kicad_sch (KiCad schematic)
At the start: 0 parts

Commit message: almost done i promise
Other:
- sheet BRUHbus ports: added none; removed Vin
- sheet Connector-Root ports: added Vin+, Vin-; removed none
Changed lines of the file:
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@@
+	(wire
+		(pts
+			(xy 186.69 57.15) (xy 181.61 57.15)
+		)
+		(stroke
+			(width 0)
+			(type default)
+		)
+	)
 	(wire
 		(pts
@@
 	(wire
 		(pts
-			(xy 82.55 83.82) (xy 82.55 102.87)
-		)
-		(stroke
-			(width 0)
-			(type default)
-		)
-	)
-	(wire
-		(pts
 			(xy 132.08 248.92) (xy 152.4 248.92)
 		)
@@
 	(wire
 		(pts
+			(xy 186.69 60.96) (xy 186.69 57.15)
+		)
+		(stroke
+			(width 0)
+			(type default)
+		)
+	)
+	(wire
+		(pts
 			(xy 132.08 237.49) (xy 152.4 237.49)
 		)
@@
 	(wire
 		(pts
-			(xy 74.93 83.82) (xy 82.55 83.82)
+			(xy 189.23 53.34) (xy 181.61 53.34)
 		)
 		(stroke
@@
 		(pts
 			(xy 132.08 199.39) (xy 152.4 199.39)
-		)
-		(stroke
-			(width 0)
-			(type default)
-		)
-	)
-	(wire
-		(pts
-			(xy 82.55 102.87) (xy 76.2 102.87)
 		)
 		(stroke
@@
 	)
 	(symbol
+		(lib_id "power:GND")
+		(at 186.69 60.96 0)
+		(unit 1)
+		(exclude_from_sim no)
+		(in_bom yes)
+		(on_board yes)
+		(dnp no)
+		(property "Reference" "#PWR025"
+			(at 186.69 67.31 0)
+			(effects
+				(font
+					(size 1.27 1.27)
+				)
+				(hide yes)
+			)
+		)
+		(property "Value" "GND"
+			(at 186.69 66.04 0)
+			(effects
+				(font
+					(size 1.27 1.27)
+				)
+			)
+		)
+		(property "Footprint" ""
+			(at 186.69 60.96 0)
+			(effects
+				(font
+					(size 1.27 1.27)
+				)
+				(hide yes)
+			)
+		)
+		(property "Datasheet" ""
+			(at 186.69 60.96 0)
+			(effects
+				(font
+					(size 1.27 1.27)
+				)
+				(hide yes)
+			)
+		)
+		(property "Description" "Power symbol creates a global label with name \"GND\" , ground"
+			(at 186.69 60.96 0)
+			(effects
+				(font
+					(size 1.27 1.27)
+				)
+				(hide yes)
+			)
+		)
+		(pin "1"
+		)
+		(instances
+			(project ""
+				(path "/4ee6c2ad-9a1b-4276-b3cf-1cc8dc52967e"
+					(reference "#PWR025")
+					(unit 1)
+				)
+			)
+		)
+	)
+	(symbol
 		(lib_id "power:+4V")
 		(at 187.96 194.31 0)
@@
 			)
 		)
+		(pin "Vin-" input
+			(at 181.61 57.15 0)
+			(effects
+				(font
+					(size 1.27 1.27)
+				)
+				(justify right)
+			)
+		)
+		(pin "Vin+" input
+			(at 181.61 53.34 0)
+			(effects
+				(font
+					(size 1.27 1.27)
+				)
+				(justify right)
+			)
+		)
 		(instances
 			(project "VCU_v1"
@@
 	)
 	(sheet
-		(at 55.88 81.28)
+		(at 189.23 45.72)
 		(size 19.05 10.16)
 		(exclude_from_sim no)
@@
 		)
 		(property "Sheetname" "Power"
-			(at 55.88 80.5684 0)
+			(at 189.23 45.0084 0)
 			(effects
 				(font
@@
 		)
 		(property "Sheetfile" "power.kicad_sch"
-			(at 55.88 92.0246 0)
+			(at 189.23 56.4646 0)
 			(effects
 				(font
@@
 		)
 		(pin "VBAT+" input
-			(at 74.93 83.82 0)
-			(effects
-				(font
-					(size 1.27 1.27)
-				)
-				(justify right)
+			(at 189.23 53.34 180)
+			(effects
+				(font
+					(size 1.27 1.27)
+				)
+				(justify left)
 			)
 		)
@@
 			(effects
 				(font
-					(size 1.27 1.27)
-				)
-				(justify right)
-			)
-		)
-		(pin "Vin" input
-			(at 76.2 102.87 0)
-			(effects
-				(font
