File: VCU_v1/pedals.kicad_sch (KiCad schematic)
At the start: 21 parts, among them U10 TSB712AIDT, U8 TSB712AIDT, U9 TSB712AIDT

Commit message: p dih r
Parts:
- removed C21, C23, C25: 100n, Capacitor_SMD:C_0603_1608Metric_Pad1.08x0.95mm_HandSolder, symbol BFR Capacitors:06035C104KAT2A
- removed R10, R14, R18: 10k, Resistor_SMD:R_0603_1608Metric_Pad0.98x0.95mm_HandSolder, symbol BFR Resistors:RMCF0603FT10K0
- removed U10: TSB712AIDT, symbol TSB712AIDT-Opamp:TSB712AIDT
- added C21, C23: 22n, Capacitor_SMD:C_0603_1608Metric_Pad1.08x0.95mm_HandSolder, symbol BFR Capacitors:VJ0603Y223KXAAC
Connections:
- net +5V: now also C21.1, C23.1
- net APPS1-2.4V: now also C20.2, R9.2; no longer U8.6 (IN2-), U8.7
- net APPS1-3.3V: now also C22.2, R13.2; no longer U9.6 (IN2-), U9.7
- net BSE-3.3V: now also C24.2, R17.2
- net GND: now also U9.5 (IN2+), C21.2, C23.2
- net at U8.5 (IN2+): now also R11.1, R12.2; no longer C20.2
- net at R15.1, R16.2: now also U9.3 (IN1+)
- net at R17.1: now also U9.1, U9.2 (IN1-)
- new net: R13.1, U8.6 (IN2-), U8.7
- new net: U9.6 (IN2-), U9.7
Other:
- moved on the sheet: C20, C22, C24, R11, R12, R13, R15, R16, R17, R7, R8, R9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

Commit message: v1 schematic (actually) complete, let the layout commence
Parts:
- added TP10, TP11, TP12, TP13, TP14, TP15: RH-5015, TestPoint:TestPoint_Keystone_5015_Micro_Mini, symbol .Test-Point:RH-5015
- U10: renamed from U9; footprint (none) -> Package_SO:SOIC-8_3.9x4.9mm_P1.27mm
- U9: renamed from U8; footprint (none) -> Package_SO:SOIC-8_3.9x4.9mm_P1.27mm
- renumbered C20 to C40, C22 to C41, C21 to C42, C23 to C43, C24 to C44, R11 to R13, R12 to R14, R7 to R15, R8 to R16, R13 to R17, R9 to R18, R15 to R19, R16 to R20, R17 to R21
Connections:
- net APPS1-2.4V: now also TP11.1
- net APPS1-3.3V: now also TP13.1
- net APPS1-IN: now also TP10.1
- net APPS2-IN: now also TP12.1
- net BSE-3.3V: now also TP15.1
- net BSE-IN: now also TP14.1

Commit message: almost done i promise
Parts:
- removed C40, C41, C44: 100n, Capacitor_SMD:C_0603_1608Metric_Pad1.08x0.95mm_HandSolder, symbol BFR Capacitors:06035C104KAT2A
- removed C42, C43: 22n, Capacitor_SMD:C_0603_1608Metric_Pad1.08x0.95mm_HandSolder, symbol BFR Capacitors:VJ0603Y223KXAAC
- removed R17, R18, R21: 10k, Resistor_SMD:R_0603_1608Metric_Pad0.98x0.95mm_HandSolder, symbol BFR Resistors:RMCF0603FT10K0
- added C1, C5: 22n, Capacitor_SMD:C_0402_1005Metric_Pad0.74x0.62mm_HandSolder, symbol BFR Capacitors:0402B223K500NT
- added C12, C40, C9: 47n, Capacitor_SMD:C_0603_1608Metric_Pad1.08x0.95mm_HandSolder, symbol BFR Capacitors:VJ0603Y473KXAAC
- added C3, C7: 100n, Capacitor_SMD:C_0603_1608Metric_Pad1.08x0.95mm_HandSolder, symbol BFR Capacitors:06035C104KAT2A
Connections:
- net +5V: now also C1.1, C3.1, C5.1, C7.1
- net APPS1-2.4V: now also U9.1, U9.2 (IN1-)
- net APPS1-3.3V: now also U9.6 (IN2-), U9.7
- net BSE-3.3V: now also U10.1, U10.2 (IN1-)
- net GND: now also C1.2, C12.2, C3.2, C40.2, C5.2, C7.2, C9.2
- net at R13.1, R14.2, U9.5 (IN2+): now also C12.1
- net at R15.1, R16.2, U9.3 (IN1+): now also C9.1
- net at R19.1, R20.2, U10.3 (IN1+): now also C40.1
Other:
- moved on the sheet: TP11, TP13, TP15
