File: VCU_v1/power.kicad_sch (KiCad schematic)
At the start: 12 parts

Commit message: almost done i promise
Other:
- sheet Buck Converters ports: added none; removed 20V-out
Changed lines of the file:
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@@
 	(wire
 		(pts
-			(xy 154.94 52.07) (xy 154.94 50.8)
+			(xy 154.94 44.45) (xy 154.94 43.18)
 		)
 		(stroke
@@
 	(wire
 		(pts
-			(xy 144.78 52.07) (xy 154.94 52.07)
+			(xy 144.78 44.45) (xy 154.94 44.45)
 		)
 		(stroke
@@
 	(wire
 		(pts
-			(xy 104.14 52.07) (xy 113.03 52.07)
+			(xy 104.14 44.45) (xy 113.03 44.45)
 		)
 		(stroke
@@
 	(wire
 		(pts
-			(xy 152.4 41.91) (xy 144.78 41.91)
+			(xy 71.12 124.46) (xy 76.2 124.46)
 		)
 		(stroke
@@
 	(wire
 		(pts
-			(xy 71.12 124.46) (xy 76.2 124.46)
+			(xy 144.78 76.2) (xy 161.29 76.2)
 		)
 		(stroke
@@
 	(wire
 		(pts
-			(xy 144.78 76.2) (xy 161.29 76.2)
+			(xy 154.94 68.58) (xy 144.78 68.58)
 		)
 		(stroke
@@
 	(wire
 		(pts
-			(xy 154.94 68.58) (xy 144.78 68.58)
+			(xy 111.76 124.46) (xy 116.84 124.46)
 		)
 		(stroke
@@
 	(wire
 		(pts
-			(xy 111.76 124.46) (xy 116.84 124.46)
+			(xy 104.14 68.58) (xy 114.3 68.58)
 		)
 		(stroke
@@
 	(wire
 		(pts
-			(xy 104.14 68.58) (xy 114.3 68.58)
+			(xy 86.36 124.46) (xy 91.44 124.46)
 		)
 		(stroke
@@
 	(wire
 		(pts
-			(xy 86.36 124.46) (xy 91.44 124.46)
-		)
-		(stroke
-			(width 0)
-			(type default)
-		)
-	)
-	(wire
-		(pts
-			(xy 152.4 38.1) (xy 152.4 41.91)
-		)
-		(stroke
-			(width 0)
-			(type default)
-		)
-	)
-	(wire
-		(pts
-			(xy 104.14 50.8) (xy 104.14 52.07)
+			(xy 104.14 43.18) (xy 104.14 44.45)
 		)
 		(stroke
@@
 	)
 	(symbol
-		(lib_id "power:VDD")
-		(at 152.4 38.1 0)
-		(unit 1)
-		(exclude_from_sim no)
-		(in_bom yes)
-		(on_board yes)
-		(dnp no)
-		(fields_autoplaced yes)
-		(property "Reference" "#PWR05"
-			(at 152.4 41.91 0)
-			(effects
-				(font
-					(size 1.27 1.27)
-				)
-				(hide yes)
-			)
-		)
-		(property "Value" "20V-AMP"
-			(at 152.4 33.02 0)
-			(effects
-				(font
-					(size 1.27 1.27)
-				)
-			)
-		)
-		(property "Footprint" ""
-			(at 152.4 38.1 0)
-			(effects
-				(font
-					(size 1.27 1.27)
-				)
-				(hide yes)
-			)
-		)
-		(property "Datasheet" ""
-			(at 152.4 38.1 0)
-			(effects
-				(font
-					(size 1.27 1.27)
-				)
-				(hide yes)
-			)
-		)
-		(property "Description" "Power symbol creates a global label with name \"VDD\""
-			(at 152.4 38.1 0)
-			(effects
-				(font
-					(size 1.27 1.27)
-				)
-				(hide yes)
-			)
-		)
-		(pin "1"
-		)
-		(instances
-			(project ""
-				(path "/4ee6c2ad-9a1b-4276-b3cf-1cc8dc52967e/9e4b5f8d-93dc-46d5-aa92-d0e0d2e07b3d"
-					(reference "#PWR05")
-					(unit 1)
-				)
-			)
-		)
-	)
-	(symbol
-		(lib_id "power:+24V")
-		(at 104.14 50.8 0)
-		(unit 1)
-		(exclude_from_sim no)
-		(in_bom yes)
-		(on_board yes)
-		(dnp no)
-		(fields_autoplaced yes)
-		(property "Reference" "#PWR03"
-			(at 104.14 54.61 0)
-			(effects
-				(font
-					(size 1.27 1.27)
-				)
-				(hide yes)
-			)
-		)
-		(property "Value" "+24V"
-			(at 104.14 45.72 0)
-			(effects
-				(font
-					(size 1.27 1.27)
-				)
-			)
-		)
-		(property "Footprint" ""
-			(at 104.14 50.8 0)
-			(effects
-				(font
-					(size 1.27 1.27)
-				)
-				(hide yes)
-			)
-		)
-		(property "Datasheet" ""
-			(at 104.14 50.8 0)
-			(effects
-				(font
-					(size 1.27 1.27)
-				)
-				(hide yes)
-			)
-		)
-		(property "Description" "Power symbol creates a global label with name \"+24V\""
-			(at 104.14 50.8 0)
-			(effects
-				(font
-					(size 1.27 1.27)
-				)
-				(hide yes)
-			)
-		)
-		(pin "1"
-		)
-		(instances
-			(project ""
-				(path "/4ee6c2ad-9a1b-4276-b3cf-1cc8dc52967e/9e4b5f8d-93dc-46d5-aa92-d0e0d2e07b3d"
-					(reference "#PWR03")
-					(unit 1)
-				)
-			)
-		)
-	)
-	(symbol
 		(lib_id ".Test-Point:RH-5015")
 		(at 101.6 124.46 0)
@@
 	)
 	(symbol
-		(lib_id "power:+24V")
+		(lib_id "power:+12V")
 		(at 152.4 95.25 0)
 		(unit 1)
@@
 		(dnp no)
 		(fields_autoplaced yes)
-		(property "Reference" "#PWR06"
+		(property "Reference" "#PWR05"
 			(at 152.4 99.06 0)
 			(effects
@@
 			)
 		)
-		(property "Value" "+24V"
+		(property "Value" "+12V"
 			(at 152.4 90.17 0)
 			(effects
@@
 			)
 		)
-		(property "Description" "Power symbol creates a global label with name \"+24V\""
+		(property "Description" "Power symbol creates a global label with name \"+12V\""
 			(at 152.4 95.25 0)
 			(effects
@@
 		)
 		(instances
-			(project "VCU_v1"
+			(project ""
 				(path "/4ee6c2ad-9a1b-4276-b3cf-1cc8dc52967e/9e4b5f8d-93dc-46d5-aa92-d0e0d2e07b3d"
-					(reference "#PWR06")
+					(reference "#PWR05")
+					(unit 1)
+				)
+			)
+		)
+	)
+	(symbol
+		(lib_id "power:+12V")
+		(at 104.14 43.18 0)
+		(unit 1)
+		(exclude_from_sim no)
+		(in_bom yes)
+		(on_board yes)
+		(dnp no)
+		(fields_autoplaced yes)
+		(property "Reference" "#PWR03"
+			(at 104.14 46.99 0)
+			(effects
+				(font
+					(size 1.27 1.27)
+				)
+				(hide yes)
+			)
+		)
+		(property "Value" "+12V"
+			(at 104.14 38.1 0)
+			(effects
+				(font
+					(size 1.27 1.27)
+				)
+			)
+		)
+		(property "Footprint" ""
+			(at 104.14 43.18 0)
+			(effects
+				(font
+					(size 1.27 1.27)
+				)
+				(hide yes)
+			)
+		)
+		(property "Datasheet" ""
+			(at 104.14 43.18 0)
+			(effects
+				(font
+					(size 1.27 1.27)
+				)
+				(hide yes)
+			)
+		)
+		(property "Description" "Power symbol creates a global label with name \"+12V\""
+			(at 104.14 43.18 0)
+			(effects
+				(font
+					(size 1.27 1.27)
+				)
+				(hide yes)
+			)
+		)
+		(pin "1"
+		)
+		(instances
+			(project ""
+				(path "/4ee6c2ad-9a1b-4276-b3cf-1cc8dc52967e/9e4b5f8d-93dc-46d5-aa92-d0e0d2e07b3d"
+					(reference "#PWR03")
 					(unit 1)
 				)
@@
 	(symbol
 		(lib_id "power:+5V")
-		(at 154.94 50.8 0)
+		(at 154.94 43.18 0)
 		(unit 1)
 		(exclude_from_sim no)
@@
 		(fields_autoplaced yes)
 		(property "Reference" "#PWR07"
-			(at 154.94 54.61 0)
+			(at 154.94 46.99 0)
 			(effects
 				(font
@@
 		)
 		(property "Value" "+5V"
-			(at 154.94 45.72 0)
+			(at 154.94 38.1 0)
 			(effects
 				(font
@@
 		)
 		(property "Footprint" ""
-			(at 154.94 50.8 0)
+			(at 154.94 43.18 0)
 			(effects
 				(font
@@
 		)
 		(property "Datasheet" ""
-			(at 154.94 50.8 0)
+			(at 154.94 43.18 0)
 			(effects
 				(font
@@
 		)
 		(property "Description" "Power symbol creates a global label with name \"+5V\""
-			(at 154.94 50.8 0)
+			(at 154.94 43.18 0)
 			(effects
 				(font
@@
 	(sheet
 		(at 113.03 34.29)
-		(size 31.75 22.86)
+		(size 31.75 15.24)
 		(exclude_from_sim no)
 		(in_bom yes)
@@
 		)
 		(property "Sheetfile" "Bucks.kicad_sch"
-			(at 113.03 57.7346 0)
+			(at 113.03 50.1146 0)
 			(effects
 				(font
@@
 		)
 		(pin "5V-out" input
-			(at 144.78 52.07 0)
+			(at 144.78 44.45 0)
 			(effects
 				(font
@@
 		)
 		(pin "BAT_FILT+" input
-			(at 113.03 52.07 180)
+			(at 113.03 44.45 180)
 			(effects
 				(font
@@
 			)
 		)
-		(pin "20V-out" input
-			(at 144.78 41.91 0)
-			(effects
-				(font
-					(size 1.27 1.27)
-				)
-				(justify right)
-			)
-		)
