File: VCU_v1/VCU_v1.kicad_pcb (KiCad board)
At the start: 4 copper layers, 217.4 x 125 mm, 271 parts, among them J1 Conn_01x04, J2 NUCLEO CONNECTOR LEFT, J3 NUCLEO CONNECTOR RIGHT, J4 Micro_SD_Card, J6 BRUHBus, J7 BRUHBus, J8 BRUHBus, Q1 PMOS, Q2 BSD235NH6327XT, Q3 SP8K80TB1, Q4 SP8K80TB1, Q5 SP8K80TB1, Q6 BSD235NH6327XT, SW1 SW_Push, U1 TPS5430, U10 TSB712AIDT, U11 MCP2562FD-E/SN, U12 MCP2562FD-E/SN, U13 TPA3116D2QDADRQ1, U14 PCM5102APWR, U2 TPS5430, U3 AMS1117-3.3, U4 MIC5200-4.8YS, U5 STM32H723ZGT6, U6 MX150 20-pin, U7 MX150 20-pin, U8 MX150 20-pin, U9 TSB712AIDT, Y1 16 MHz, Y2 32.768 kHz

Commit message: aughhhh
Parts:
- added R33: 0, Resistor_SMD:R_0805_2012Metric_Pad1.20x1.40mm_HandSolder, F.Cu at (231.6, 162.6)
- added R35: 0, Resistor_SMD:R_0805_2012Metric_Pad1.20x1.40mm_HandSolder, F.Cu at (43.9, 83.7)
- added R37: 0, Resistor_SMD:R_0805_2012Metric_Pad1.20x1.40mm_HandSolder, F.Cu at (43.7, 102.2)
- moved TP28 11.9 mm to (156.8, 68.6)
- moved TP40 11.4 mm to (185.5, 66.2)
- moved TP32 6.50 mm to (169.4, 68.5)
- moved TP30 5.91 mm to (163.2, 68.6)
- moved R41 4.42 mm to (90.9, 84.7), turned to 0 degrees
- moved TP22 3.30 mm to (92.8, 103.4)
- moved TP23 2.80 mm to (92.8, 100.3)
- moved TP41 2.67 mm to (199.4, 66.2)
- moved R58 2.50 mm to (65.3, 65.3)
- moved R64 2.49 mm to (62.5, 74.3)
- moved R59 2.46 mm to (62.9, 65.3)
- moved R63 2.29 mm to (64.8, 74.3)
- moved R71 1.76 mm to (193.0, 65.4)
- moved R78 1.67 mm to (48.9, 79.0)
- moved R65 1.59 mm to (192.9, 67.3)
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Connections:
- J6 pad SH: unconnected-(J6-SHIELD-PadSH) -> Net-(J6-SHIELD)
- J7 pad SH: unconnected-(J7-SHIELD-PadSH) -> Net-(J7-SHIELD)
- J8 pad SH: unconnected-(J8-SHIELD-PadSH) -> Net-(J8-SHIELD)
Routing:
- net /STM32-Root/STM32H723ZGT6/PB5: track 0.00 -> 251.7 mm, vias 0 -> 3
- net /Connector-Root/IMD-FAULT: track 0.00 -> 222.6 mm, vias 0 -> 1
- net /Connector-Root/BMS-FAULT: track 0.00 -> 216.0 mm, vias 0 -> 1
- net /Connector-Root/BRAKE_LIGHT: track 0.00 -> 170.3 mm, vias 0 -> 1
- net /Connector-Root/BSPD-FAULT: track 0.00 -> 168.6 mm, vias 0 -> 2
- net /Connector-Root/BSPD_FAULT+: track 0.00 -> 162.7 mm, vias 0 -> 2
- net /BRUHbus/CAN1_H: track 0.00 -> 132.8 mm, vias 0 -> 3
- net /BRUHbus/CAN1_L: track 0.00 -> 125.7 mm, vias 0 -> 2
- net GND: track 45.9 -> 151.4 mm, vias 85 -> 136
- net /STM32-Root/STM32H723ZGT6/PB6: track 0.00 -> 78.3 mm, vias 0 -> 2
- net +3.3V: track 45.2 -> 102.3 mm, vias 54 -> 73
- net /BRUHbus/CAN2_L: track 0.00 -> 55.8 mm, vias 0 -> 1
- net /STM32-Root/STM32H723ZGT6/PD1: track 0.00 -> 52.0 mm, vias 0 -> 2
- net /BRUHbus/CAN2_H: track 0.00 -> 49.8 mm
- net /STM32-Root/STM32H723ZGT6/PD0: track 0.00 -> 49.4 mm, vias 0 -> 2
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- added copper zone on F.Cu, net +4.8V

Commit message: almost done i promise
Parts:
- removed C41, C44: 100n, Capacitor_SMD:C_0603_1608Metric_Pad1.08x0.95mm_HandSolder
- removed C42, C43: 22n, Capacitor_SMD:C_0603_1608Metric_Pad1.08x0.95mm_HandSolder
- removed D1: B340LA-13-F, Diode_SMD:D_SMA_Handsoldering
- removed D3: GREEN LED, LED_SMD:LED_0603_1608Metric_Pad1.05x0.95mm_HandSolder
- removed L1: 33u, SER2211-333MED:Untitled
- removed R40, R57, R65, R71, R79, R80, R81, R82: 1.6k, Resistor_SMD:R_0603_1608Metric_Pad0.98x0.95mm_HandSolder
- removed TP2: RH-5015, TestPoint:TestPoint_Keystone_5015_Micro_Mini
- removed U1: TPS5430, TPS5430DDAR:Untitled
- added R39: 2.4k, Resistor_SMD:R_0603_1608Metric_Pad0.98x0.95mm_HandSolder, F.Cu at (-7.11, 82.0)
- C1: value 100u -> 22n; footprint Capacitor_THT:CP_Radial_D8.0mm_P3.50mm -> Capacitor_SMD:C_0402_1005Metric_Pad0.74x0.62mm_HandSolder
- C12: value 150u -> 47n; footprint Capacitor_THT:CP_Radial_D8.0mm_P3.50mm -> Capacitor_SMD:C_0603_1608Metric_Pad1.08x0.95mm_HandSolder
- C3: value 10u -> 100n
- C40: value 100n -> 47n
- C5: value 10u -> 22n; footprint Capacitor_SMD:C_0603_1608Metric_Pad1.08x0.95mm_HandSolder -> Capacitor_SMD:C_0402_1005Metric_Pad0.74x0.62mm_HandSolder
- C7: value 10n -> 100n
- C9: value 220p -> 47n
- R1: value 56 -> 1.0k
- R12, R38: value 1.6k -> 2.4k
- R17, R18, R21, R3: value 10k -> 2.4k
- R4: value 620 -> 2.4k
- R7, R8: value 220 -> 2.4k
- moved R38 247.7 mm to (-10.5, 75.1)
- moved R17 162.7 mm to (223.8, 155.6), turned to 90 degrees
- moved C5 139.4 mm to (74.9, 75.7), turned to 90 degrees
- moved C1 135.4 mm to (87.1, 72.9), turned to 0 degrees
- moved C12 134.4 mm to (81.5, 68.1), turned to 180 degrees
- moved C3 130.2 mm to (87.6, 74.4), turned to 0 degrees
- moved C7 127.2 mm to (76.5, 75.8), turned to 90 degrees
- moved R4 120.5 mm to (317.5, 115.1)
- moved TP49 120.1 mm to (323.8, 116.2)
- moved C9 114.3 mm to (96.8, 67.3), turned to 0 degrees
- moved R18 90.1 mm to (2.33, 78.3)
- moved R21 80.5 mm to (-4.57, 70.1)
- moved R8 59.7 mm to (196.1, 68.6)
- moved R7 59.3 mm to (191.9, 67.3)
- moved R12 47.1 mm to (224.3, 147.6), turned to 90 degrees
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Connections:
- C1 pad 1: +24V -> +5V
- C12 pad 1: 20V-AMP -> Net-(U9B-IN2+)
- C2 pad 1: +24V -> +12V
- C3 pad 1: +24V -> +5V
- C4 pad 1: +24V -> +12V
- C40 pad 1: GND -> Net-(U10A-IN1+)
- C40 pad 2: /STM32-Root/STM32H723ZGT6/PC2 -> GND
- C45 pad 2: Net-(U11-STDBY) -> GND
- C46 pad 2: Net-(U12-STDBY) -> GND
- C5 pad 1: +24V -> +5V
- C50 pad 1: 20V-AMP -> +12V
- C55 pad 1: 20V-AMP -> +12V
- C56 pad 1: 20V-AMP -> +12V
- C6 pad 1: +24V -> +12V
- C62 pad 1: 20V-AMP -> +12V
- C63 pad 1: 20V-AMP -> +12V
- C65 pad 1: 20V-AMP -> +12V
- C66 pad 1: 20V-AMP -> +12V
- C7 pad 1: Net-(D1-K) -> +5V
- C7 pad 2: Net-(U1-BOOT) -> GND
- C9 pad 1: Net-(D1-K) -> Net-(U9A-IN1+)
- C9 pad 2: Net-(C9-Pad2) -> GND
- D5 pad 1: +24V -> +12V
- D6 pad 2: +24V -> +12V
- J6 pad 3: GND -> unconnected-(J6--Vs-Pad3)
- J6 pad 4: /BRUHbus/Vin -> Net-(J6-+Vs-Pad4)
- J6 pad 5: /BRUHbus/Vin -> Net-(J6-+Vs-Pad4)
- J6 pad 6: GND -> unconnected-(J6--Vs-Pad6)
- J7 pad 4: +24V -> +12V
- J7 pad 5: +24V -> +12V
- J8 pad 4: +24V -> +12V
- J8 pad 5: +24V -> +12V
- Q1 pad 1: /BRUHbus/Vin -> /Connector-Root/Vin+
- Q1 pad 3: +24V -> +12V
- R1 pad 1: Net-(C9-Pad2) -> Net-(D4-A)
- R1 pad 2: GND -> +5V
- R12 pad 1: Net-(D7-A) -> Net-(J6-+Vs-Pad4)
- R12 pad 2: +24V -> Net-(J6-POWER_GOOD)
- R17 pad 1: Net-(U9B-IN2-) -> Net-(J6-CAN_IND)
- R17 pad 2: /STM32-Root/STM32H723ZGT6/PF10 -> +12V
- R18 pad 1: Net-(U9A-IN1-) -> +12V
- R18 pad 2: /STM32-Root/STM32H723ZGT6/PC2 -> Net-(J7-POWER_GOOD)
- R21 pad 1: Net-(U10A-IN1-) -> +12V
- R21 pad 2: /STM32-Root/STM32H723ZGT6/PF8 -> Net-(J8-POWER_GOOD)
- R22 pad 2: 20V-AMP -> +12V
- R25 pad 2: 20V-AMP -> +12V
- R3 pad 1: Net-(U1-VSENSE) -> Net-(D7-A)
- R3 pad 2: 20V-AMP -> +12V
- R38 pad 1: Net-(J6-CAN_IND) -> Net-(J7-CAN_IND)
- R38 pad 2: +24V -> +12V
- R4 pad 1: GND -> /Connector-Root/BSPD_FAULT+
- R4 pad 2: Net-(U1-VSENSE) -> +12V
- R7 pad 1: Net-(D3-A) -> /Connector-Root/BMS_FAULT+
- R7 pad 2: 20V-AMP -> +12V
- R8 pad 1: Net-(D4-A) -> +12V
- R8 pad 2: +5V -> /Connector-Root/IMD_FAULT+
- TP5 pad 1: +24V -> +12V
- TP6 pad 1: /BRUHbus/Vin -> /Connector-Root/Vin+
- U10 pad 1: Net-(U10A-IN1-) -> /STM32-Root/STM32H723ZGT6/PF8
- U10 pad 2: Net-(U10A-IN1-) -> /STM32-Root/STM32H723ZGT6/PF8
- U11 pad 8: Net-(U11-STDBY) -> GND
- U12 pad 8: Net-(U12-STDBY) -> GND
- U13 pad 17: 20V-AMP -> +12V
- U13 pad 18: 20V-AMP -> +12V
- U13 pad 19: 20V-AMP -> +12V
- U13 pad 31: 20V-AMP -> +12V
- U13 pad 32: 20V-AMP -> +12V
- U2 pad 7: +24V -> +12V
- U6 pad 17: unconnected-(U6-Pad17) -> /STM32-Root/STM32H723ZGT6/PB15
- U6 pad 7: unconnected-(U6-Pad7) -> /STM32-Root/STM32H723ZGT6/PG4
- U7 pad 1: /STM32-Root/STM32H723ZGT6/PG4 -> /Connector-Root/Vin+
- U7 pad 11: /STM32-Root/STM32H723ZGT6/PB15 -> GND
- U7 pad 12: /STM32-Root/STM32H723ZGT6/PG9 -> /STM32-Root/STM32H723ZGT6/PG15
- U7 pad 13: /STM32-Root/STM32H723ZGT6/PG10 -> /STM32-Root/STM32H723ZGT6/PG13
- U7 pad 15: /STM32-Root/STM32H723ZGT6/PG12 -> /STM32-Root/STM32H723ZGT6/PG9
- U7 pad 16: /STM32-Root/STM32H723ZGT6/PG13 -> /STM32-Root/STM32H723ZGT6/PG8
- U7 pad 17: /STM32-Root/STM32H723ZGT6/PG14 -> /STM32-Root/STM32H723ZGT6/PG7
- U7 pad 18: /STM32-Root/STM32H723ZGT6/PG15 -> /STM32-Root/STM32H723ZGT6/PG6
- U7 pad 2: /STM32-Root/STM32H723ZGT6/PG5 -> /STM32-Root/STM32H723ZGT6/PG12
- U7 pad 3: /STM32-Root/STM32H723ZGT6/PG6 -> /STM32-Root/STM32H723ZGT6/PG14
- U7 pad 4: /STM32-Root/STM32H723ZGT6/PG7 -> /STM32-Root/STM32H723ZGT6/PG10
- U7 pad 5: /STM32-Root/STM32H723ZGT6/PG8 -> /STM32-Root/STM32H723ZGT6/PG5
- U8 pad 15: /STM32-Root/STM32H723ZGT6/PA0 -> /STM32-Root/STM32H723ZGT6/PA2
- U8 pad 17: /STM32-Root/STM32H723ZGT6/PA2 -> /STM32-Root/STM32H723ZGT6/PA0
- U9 pad 1: Net-(U9A-IN1-) -> /STM32-Root/STM32H723ZGT6/PC2
- U9 pad 2: Net-(U9A-IN1-) -> /STM32-Root/STM32H723ZGT6/PC2
- U9 pad 6: Net-(U9B-IN2-) -> /STM32-Root/STM32H723ZGT6/PF10
- U9 pad 7: Net-(U9B-IN2-) -> /STM32-Root/STM32H723ZGT6/PF10
Routing:
- net /STM32-Root/STM32H723ZGT6/PA0: track 0.00 -> 243.5 mm
- net /STM32-Root/STM32H723ZGT6/PA1: track 0.00 -> 240.9 mm
- net /STM32-Root/STM32H723ZGT6/PA2: track 0.00 -> 240.5 mm
- net /STM32-Root/STM32H723ZGT6/PG1: track 0.00 -> 211.1 mm, vias 0 -> 2
- net /STM32-Root/STM32H723ZGT6/PG0: track 0.00 -> 210.0 mm, vias 0 -> 2
- net /STM32-Root/STM32H723ZGT6/PG2: track 0.00 -> 199.7 mm, vias 0 -> 3
- net /STM32-Root/STM32H723ZGT6/PG3: track 0.00 -> 198.6 mm, vias 0 -> 3
- net /STM32-Root/STM32H723ZGT6/PG9: track 0.00 -> 194.0 mm, vias 0 -> 1
- net /STM32-Root/STM32H723ZGT6/PG5: track 0.00 -> 178.9 mm, vias 0 -> 1
- net /STM32-Root/STM32H723ZGT6/PC2: track 1.80 -> 119.3 mm
- net /STM32-Root/STM32H723ZGT6/PF10: track 3.47 -> 114.6 mm
- net /STM32-Root/STM32H723ZGT6/PF8: track 1.80 -> 100.6 mm
- net /STM32-Root/STM32H723ZGT6/PB15: track 0.00 -> 82.2 mm, vias 0 -> 1
- net /STM32-Root/STM32H723ZGT6/PG4: track 0.00 -> 76.1 mm, vias 0 -> 1
- net /STM32-Root/STM32H723ZGT6/VBAT: track 0.00 -> 74.0 mm
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- added copper zone on F.Cu, net +12V
- added copper zone on In2.Cu, net +12V
- added copper zone on B.Cu, net /Connector-Root/Vin+
- added copper zone on F.Cu, net /Connector-Root/Vin+
- removed copper zone on F.Cu, net +24V
- removed copper zone on In2.Cu, net +24V
- removed copper zone on F.Cu, net /BRUHbus/Vin
- removed copper zone on F.Cu, net 20V-AMP
- removed copper zone on In2.Cu, net 20V-AMP
- removed copper zone on F.Cu, net Net-(D1-K)

Commit message: fixing drc errors, done besides that
Parts:
- removed U4: MIC5200-4.8YS, Package_TO_SOT_SMD:SOT-223-3_TabPin2
- added U1: XC6221B481MR-G, Package_TO_SOT_SMD:SOT-23-5, F.Cu at (51.4, 69.2)
- moved R4 234.0 mm to (83.8, 126.5)
- moved TP49 86.4 mm to (238.8, 101.1)
- moved R21 55.5 mm to (43.7, 97.5), turned to -90 degrees
- moved R38 54.4 mm to (43.6, 68.8), turned to -90 degrees
- moved R39 51.3 mm to (43.8, 88.5), turned to -90 degrees
- moved R18 41.4 mm to (43.7, 76.6)
- moved R28 6.01 mm to (132.0, 64.8), turned to -90 degrees
- moved C74 5.02 mm to (132.0, 68.7), turned to 90 degrees
- moved C68 3.48 mm to (135.1, 70.1), turned to 90 degrees
- moved C70 2.56 mm to (135.5, 67.2)
- moved R24 1.71 mm to (129.2, 99.3)
- moved R23 1.71 mm to (125.6, 99.3)
- moved R37 1.44 mm to (44.7, 103.3), turned to 180 degrees
- moved TP25 0.90 mm to (122.7, 67.4)
- moved TP26 0.74 mm to (128.3, 67.3)
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Connections:
- J2 pad 11: /STM32-Root/STM32H723ZGT6/PF7 -> unconnected-(J2-Pin_11-Pad11)
- J2 pad 13: /STM32-Root/STM32H723ZGT6/PA13 -> unconnected-(J2-Pin_13-Pad13)
- J2 pad 15: /STM32-Root/STM32H723ZGT6/PA14 -> unconnected-(J2-Pin_15-Pad15)
- J2 pad 17: /STM32-Root/STM32H723ZGT6/PA15 -> unconnected-(J2-Pin_17-Pad17)
- J2 pad 21: /STM32-Root/STM32H723ZGT6/PB7 -> unconnected-(J2-Pin_21-Pad21)
- J2 pad 23: /STM32-Root/STM32H723ZGT6/PC13 -> unconnected-(J2-Pin_23-Pad23)
- J2 pad 25: /STM32-Root/STM32H723ZGT6/PC14 -> unconnected-(J2-Pin_25-Pad25)
- J2 pad 27: /STM32-Root/STM32H723ZGT6/PC15 -> unconnected-(J2-Pin_27-Pad27)
- J2 pad 32: /STM32-Root/STM32H723ZGT6/PA4 -> unconnected-(J2-Pin_32-Pad32)
- J2 pad 34: /STM32-Root/STM32H723ZGT6/PB0 -> unconnected-(J2-Pin_34-Pad34)
- J2 pad 37: /STM32-Root/STM32H723ZGT6/PC3 -> unconnected-(J2-Pin_37-Pad37)
- J2 pad 38: /STM32-Root/STM32H723ZGT6/PC0 -> unconnected-(J2-Pin_38-Pad38)
- J2 pad 39: /STM32-Root/STM32H723ZGT6/PD4 -> unconnected-(J2-Pin_39-Pad39)
- J2 pad 40: /STM32-Root/STM32H723ZGT6/PD3 -> unconnected-(J2-Pin_40-Pad40)
- J2 pad 41: /STM32-Root/STM32H723ZGT6/PD5 -> unconnected-(J2-Pin_41-Pad41)
- J2 pad 42: /STM32-Root/STM32H723ZGT6/PG2 -> unconnected-(J2-Pin_42-Pad42)
- J2 pad 43: /STM32-Root/STM32H723ZGT6/PD6 -> unconnected-(J2-Pin_43-Pad43)
- J2 pad 44: /STM32-Root/STM32H723ZGT6/PG3 -> unconnected-(J2-Pin_44-Pad44)
- J2 pad 45: /STM32-Root/STM32H723ZGT6/PD7 -> unconnected-(J2-Pin_45-Pad45)
- J2 pad 46: /STM32-Root/STM32H723ZGT6/PE2 -> unconnected-(J2-Pin_46-Pad46)
- J2 pad 47: /STM32-Root/STM32H723ZGT6/PE3 -> unconnected-(J2-Pin_47-Pad47)
- J2 pad 48: /STM32-Root/STM32H723ZGT6/PE4 -> unconnected-(J2-Pin_48-Pad48)
- J2 pad 50: /STM32-Root/STM32H723ZGT6/PE5 -> unconnected-(J2-Pin_50-Pad50)
- J2 pad 51: /STM32-Root/STM32H723ZGT6/PF1 -> unconnected-(J2-Pin_51-Pad51)
- J2 pad 52: /STM32-Root/STM32H723ZGT6/PF2 -> unconnected-(J2-Pin_52-Pad52)
- J2 pad 53: /STM32-Root/STM32H723ZGT6/PF0 -> unconnected-(J2-Pin_53-Pad53)
- J2 pad 56: /STM32-Root/STM32H723ZGT6/PF9 -> unconnected-(J2-Pin_56-Pad56)
- J2 pad 58: /STM32-Root/STM32H723ZGT6/PG1 -> unconnected-(J2-Pin_58-Pad58)
- J2 pad 59: /STM32-Root/STM32H723ZGT6/PG0 -> unconnected-(J2-Pin_59-Pad59)
- J2 pad 61: /STM32-Root/STM32H723ZGT6/PE1 -> unconnected-(J2-Pin_61-Pad61)
- J2 pad 62: /STM32-Root/STM32H723ZGT6/PE6 -> unconnected-(J2-Pin_62-Pad62)
- J2 pad 63: /STM32-Root/STM32H723ZGT6/PG9 -> unconnected-(J2-Pin_63-Pad63)
- J2 pad 64: /STM32-Root/STM32H723ZGT6/PG15 -> unconnected-(J2-Pin_64-Pad64)
- J2 pad 65: /STM32-Root/STM32H723ZGT6/PG12 -> unconnected-(J2-Pin_65-Pad65)
- J2 pad 66: /STM32-Root/STM32H723ZGT6/PG10 -> unconnected-(J2-Pin_66-Pad66)
- J2 pad 68: /STM32-Root/STM32H723ZGT6/PG13 -> unconnected-(J2-Pin_68-Pad68)
- J2 pad 69: /STM32-Root/STM32H723ZGT6/PD9 -> unconnected-(J2-Pin_69-Pad69)
- J2 pad 70: /STM32-Root/STM32H723ZGT6/PG11 -> unconnected-(J2-Pin_70-Pad70)
- J2 pad 9: /STM32-Root/STM32H723ZGT6/PF6 -> unconnected-(J2-Pin_9-Pad9)
- J3 pad 10: /STM32-Root/STM32H723ZGT6/PD8 -> unconnected-(J3-Pin_10-Pad10)
- J3 pad 12: /STM32-Root/STM32H723ZGT6/PA12 -> unconnected-(J3-Pin_12-Pad12)
- J3 pad 14: /STM32-Root/STM32H723ZGT6/PA11 -> unconnected-(J3-Pin_14-Pad14)
- J3 pad 18: /STM32-Root/STM32H723ZGT6/PB11 -> unconnected-(J3-Pin_18-Pad18)
- J3 pad 19: /STM32-Root/STM32H723ZGT6/PC7 -> unconnected-(J3-Pin_19-Pad19)
- J3 pad 2: /STM32-Root/STM32H723ZGT6/PC8 -> unconnected-(J3-Pin_2-Pad2)
- J3 pad 21: /STM32-Root/STM32H723ZGT6/PA9 -> unconnected-(J3-Pin_21-Pad21)
- J3 pad 22: /STM32-Root/STM32H723ZGT6/PB2 -> unconnected-(J3-Pin_22-Pad22)
- J3 pad 23: /STM32-Root/STM32H723ZGT6/PA8 -> unconnected-(J3-Pin_23-Pad23)
- J3 pad 24: /STM32-Root/STM32H723ZGT6/PB1 -> unconnected-(J3-Pin_24-Pad24)
- J3 pad 27: /STM32-Root/STM32H723ZGT6/PB4 -> unconnected-(J3-Pin_27-Pad27)
- J3 pad 28: /STM32-Root/STM32H723ZGT6/PB14 -> unconnected-(J3-Pin_28-Pad28)
- J3 pad 3: /STM32-Root/STM32H723ZGT6/PB8 -> unconnected-(J3-Pin_3-Pad3)
- J3 pad 31: /STM32-Root/STM32H723ZGT6/PB3 -> unconnected-(J3-Pin_31-Pad31)
- J3 pad 33: /STM32-Root/STM32H723ZGT6/PA10 -> unconnected-(J3-Pin_33-Pad33)
- J3 pad 34: /STM32-Root/STM32H723ZGT6/PC4 -> unconnected-(J3-Pin_34-Pad34)
- J3 pad 36: /STM32-Root/STM32H723ZGT6/PF5 -> unconnected-(J3-Pin_36-Pad36)
- J3 pad 37: /STM32-Root/STM32H723ZGT6/PA3 -> unconnected-(J3-Pin_37-Pad37)
- J3 pad 38: /STM32-Root/STM32H723ZGT6/PF4 -> unconnected-(J3-Pin_38-Pad38)
- J3 pad 4: /STM32-Root/STM32H723ZGT6/PC6 -> unconnected-(J3-Pin_4-Pad4)
- J3 pad 41: /STM32-Root/STM32H723ZGT6/PD13 -> unconnected-(J3-Pin_41-Pad41)
- J3 pad 43: /STM32-Root/STM32H723ZGT6/PD12 -> unconnected-(J3-Pin_43-Pad43)
- J3 pad 45: /STM32-Root/STM32H723ZGT6/PD11 -> unconnected-(J3-Pin_45-Pad45)
- J3 pad 46: /STM32-Root/STM32H723ZGT6/PD14 -> unconnected-(J3-Pin_46-Pad46)
- J3 pad 47: /STM32-Root/STM32H723ZGT6/PE10 -> unconnected-(J3-Pin_47-Pad47)
- J3 pad 48: /STM32-Root/STM32H723ZGT6/PD15 -> unconnected-(J3-Pin_48-Pad48)
- J3 pad 49: /STM32-Root/STM32H723ZGT6/PE12 -> unconnected-(J3-Pin_49-Pad49)
- J3 pad 5: /STM32-Root/STM32H723ZGT6/PB9 -> unconnected-(J3-Pin_5-Pad5)
- J3 pad 51: /STM32-Root/STM32H723ZGT6/PE14 -> unconnected-(J3-Pin_51-Pad51)
- J3 pad 53: /STM32-Root/STM32H723ZGT6/PE15 -> unconnected-(J3-Pin_53-Pad53)
- J3 pad 55: /STM32-Root/STM32H723ZGT6/PE13 -> unconnected-(J3-Pin_55-Pad55)
- J3 pad 56: /STM32-Root/STM32H723ZGT6/PE11 -> unconnected-(J3-Pin_56-Pad56)
- J3 pad 57: /STM32-Root/STM32H723ZGT6/PF13 -> unconnected-(J3-Pin_57-Pad57)
- J3 pad 58: /STM32-Root/STM32H723ZGT6/PF3 -> unconnected-(J3-Pin_58-Pad58)
- J3 pad 59: /STM32-Root/STM32H723ZGT6/PF12 -> unconnected-(J3-Pin_59-Pad59)
- J3 pad 6: /STM32-Root/STM32H723ZGT6/PC5 -> unconnected-(J3-Pin_6-Pad6)
- J3 pad 61: /STM32-Root/STM32H723ZGT6/PG14 -> unconnected-(J3-Pin_61-Pad61)
- J3 pad 62: /STM32-Root/STM32H723ZGT6/PF11 -> unconnected-(J3-Pin_62-Pad62)
- J3 pad 64: /STM32-Root/STM32H723ZGT6/PE0 -> unconnected-(J3-Pin_64-Pad64)
- J3 pad 65: /STM32-Root/STM32H723ZGT6/PD10 -> unconnected-(J3-Pin_65-Pad65)
- J3 pad 66: /STM32-Root/STM32H723ZGT6/PG8 -> unconnected-(J3-Pin_66-Pad66)
- J3 pad 67: /STM32-Root/STM32H723ZGT6/PG7 -> unconnected-(J3-Pin_67-Pad67)
- J3 pad 68: /STM32-Root/STM32H723ZGT6/PG5 -> unconnected-(J3-Pin_68-Pad68)
- J3 pad 69: /STM32-Root/STM32H723ZGT6/PG4 -> unconnected-(J3-Pin_69-Pad69)
- J3 pad 70: /STM32-Root/STM32H723ZGT6/PG6 -> unconnected-(J3-Pin_70-Pad70)
- U7 pad 15: /STM32-Root/STM32H723ZGT6/PG9 -> /STM32-Root/STM32H723ZGT6/PG10
- U7 pad 2: /STM32-Root/STM32H723ZGT6/PG12 -> /STM32-Root/STM32H723ZGT6/PG14
- U7 pad 3: /STM32-Root/STM32H723ZGT6/PG14 -> /STM32-Root/STM32H723ZGT6/PG12
- U7 pad 4: /STM32-Root/STM32H723ZGT6/PG10 -> /STM32-Root/STM32H723ZGT6/PG9
Routing:
- net /BRUHbus/CAN2_L: track 55.3 -> 302.4 mm, vias 1 -> 3
- net /BRUHbus/CAN2_H: track 49.8 -> 295.9 mm, vias 0 -> 2
- net /STM32-Root/STM32H723ZGT6/PB12: track 0.00 -> 215.6 mm, vias 0 -> 2
- net /STM32-Root/STM32H723ZGT6/PG15: track 0.00 -> 198.0 mm, vias 0 -> 1
- net /STM32-Root/STM32H723ZGT6/PG10: track 0.00 -> 195.4 mm, vias 0 -> 1
- net /STM32-Root/STM32H723ZGT6/PG13: track 0.00 -> 195.0 mm, vias 0 -> 1
- net /STM32-Root/STM32H723ZGT6/PG11: track 0.00 -> 194.1 mm, vias 0 -> 1
- net /STM32-Root/STM32H723ZGT6/PG14: track 0.00 -> 192.8 mm, vias 0 -> 1
- net /STM32-Root/STM32H723ZGT6/PC1: track 0.00 -> 191.6 mm, vias 0 -> 3
- net /STM32-Root/STM32H723ZGT6/PG6: track 0.00 -> 190.4 mm, vias 0 -> 1
- net /STM32-Root/STM32H723ZGT6/PG12: track 0.12 -> 190.3 mm, vias 0 -> 1
- net /STM32-Root/STM32H723ZGT6/PG7: track 0.00 -> 189.5 mm, vias 0 -> 1
- net /STM32-Root/STM32H723ZGT6/PG8: track 0.00 -> 188.4 mm, vias 0 -> 1
- net /STM32-Root/STM32H723ZGT6/PE11: track 0.00 -> 183.6 mm, vias 0 -> 1
- net /STM32-Root/STM32H723ZGT6/PE10: track 0.00 -> 180.4 mm, vias 0 -> 1
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- added copper zone on F.Cu, net /Connector-Root/SPEAKER+
- added copper zone on F.Cu, net /Connector-Root/SPEAKER-
Other:
- copper layers 4 -> 6
