File: VCU_v1/VCU_v1.kicad_pcb (KiCad board)
At the start: 6 copper layers, 217.4 x 125 mm, 258 parts, among them J1 Conn_01x04, J2 NUCLEO CONNECTOR LEFT, J3 NUCLEO CONNECTOR RIGHT, J4 Micro_SD_Card, J6 BRUHBus, J7 BRUHBus, J8 BRUHBus, Q1 PMOS, Q2 BSD235NH6327XT, Q3 SP8K80TB1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

Commit message: full v1 board, ordered
Routing:
- net +3.3V: track 106.5 -> 111.1 mm, vias 75 -> 77
- net GND: track 237.6 -> 237.2 mm, vias 177 -> 191
- net /STM32-Root/STM32H723ZGT6/PE7: vias 2 -> 3
