File: VCU_v2/BRUHbus.kicad_sch (KiCad schematic)
At the start: 22 parts, among them J3 BRUHBus, J4 BRUHBus, J5 BRUHBus, Q2 BSD235NH6327XT, Q3 BSD235NH6327XT

Commit message: placements friggin 80% friggin done shoutout epstein
Parts:
- renumbered J3 to J6, J4 to J7, J5 to J8, Q3 to Q6, R30 to R12, R29 to R17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

Commit message: vcu v2 schematics done
Parts:
- renumbered J6 to J3, J7 to J4, J8 to J5, Q6 to Q3, R34 to R27, R36 to R28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
