File: VCU_v2/rtd_audio.kicad_sch (KiCad schematic)
At the start: 52 parts, among them U12 TPA3116D2QDADRQ1, U13 PCM5102APWR

Commit message: placements friggin 80% friggin done shoutout epstein
Parts:
- renumbered C43 to C47, C44 to C48, C45 to C49, C46 to C50, C47 to C51, C48 to C52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

Commit message: vcu v2 schematics done
Parts:
- renumbered C47 to C43, C48 to C44, C49 to C45, C50 to C46, C51 to C47, C52 to C48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
