File: VCU_v2/dash_ext_int.kicad_sch (KiCad schematic)
At the start: 55 parts, among them Q3 SP8K80TB1, Q4 SP8K80TB1, Q5 SP8K80TB1

Commit message: vcu v2 schematics done
Parts:
- renumbered C81 to C77, C82 to C78, C83 to C79, C84 to C80, D8 to D6, Q3 to Q4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

Commit message: placements friggin 80% friggin done shoutout epstein
Parts:
- renumbered C77 to C81, C78 to C82, C79 to C83, C80 to C84, D6 to D8, Q4 to Q3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
