File: VCU_v2/pedals.kicad_sch (KiCad schematic)
At the start: 21 parts, among them U10 TSB712AIDT, U9 TSB712AIDT

Commit message: vcu v2 schematics done
Parts:
- renumbered C12 to C34, C9 to C35, C1 to C36, C40 to C37, C3 to C38, C5 to C39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

Commit message: placements friggin 80% friggin done shoutout epstein
Parts:
- renumbered C36 to C1, C34 to C12, C38 to C3, C37 to C40, C39 to C5, C40 to C7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
