File: VCU_v2/VCU_v2.kicad_pcb (KiCad board)
At the start: 6 copper layers, 217.4 x 125 mm, 258 parts, among them J1 Conn_01x04, J2 NUCLEO CONNECTOR LEFT, J3 NUCLEO CONNECTOR RIGHT, J4 Micro_SD_Card, J6 BRUHBus, J7 BRUHBus, J8 BRUHBus, Q1 PMOS, Q2 BSD235NH6327XT, Q3 SP8K80TB1, Q4 SP8K80TB1, Q5 SP8K80TB1, Q6 BSD235NH6327XT, SW1 SW_Push, U1 XC6221B481MR-G, U10 TSB712AIDT, U11 MCP2562FD-E/SN, U12 MCP2562FD-E/SN, U13 TPA3116D2QDADRQ1, U14 PCM5102APWR, U2 TPS5430, U3 AMS1117-3.3, U5 STM32H723ZGT6, U6 MX150 20-pin, U7 MX150 20-pin, U8 MX150 20-pin, U9 TSB712AIDT, Y1 16 MHz, Y2 32.768 kHz

Commit message: placements friggin 80% friggin done shoutout epstein
Parts:
- removed J2: NUCLEO CONNECTOR LEFT, Connector_PinHeader_2.54mm:PinHeader_2x35_P2.54mm_Vertical
- removed J3: NUCLEO CONNECTOR RIGHT, Connector_PinHeader_2.54mm:PinHeader_2x35_P2.54mm_Vertical
- removed JP2: Jumper_3_Open, Connector_PinHeader_2.54mm:PinHeader_1x03_P2.54mm_Vertical
- removed R41: 120, Resistor_SMD:R_0603_1608Metric_Pad0.98x0.95mm_HandSolder
- removed U6, U7, U8: MX150 20-pin, 20pinMX150Header:CONN_SD-34829-001_20_ST_MOL
- added C41: 100nF, Capacitor_SMD:C_0603_1608Metric_Pad1.08x0.95mm_HandSolder, F.Cu at (151.8, -34.2)
- added C42: 100nF, Capacitor_SMD:C_0603_1608Metric_Pad1.08x0.95mm_HandSolder, F.Cu at (151.8, -31.7)
- added C44: 100nF, Capacitor_SMD:C_0603_1608Metric_Pad1.08x0.95mm_HandSolder, F.Cu at (151.8, -29.1)
- added C86: 100nF, Capacitor_SMD:C_0603_1608Metric_Pad1.08x0.95mm_HandSolder, F.Cu at (151.8, -26.6)
- added D1: BZT52C16, Diode_SMD:D_SOD-123, F.Cu at (170.2, -16.2)
- added D12: BZT52C16, Diode_SMD:D_SOD-123, F.Cu at (170.2, -12.8)
- added D13: Red, LED_SMD:LED_0805_2012Metric, F.Cu at (151.8, -16.3)
- added D14: Red, LED_SMD:LED_0805_2012Metric, F.Cu at (151.8, -13.3)
- added D15: BZT52C16, Diode_SMD:D_SOD-123, F.Cu at (170.2, -9.48)
- added D16: Red, LED_SMD:LED_0805_2012Metric, F.Cu at (151.8, -10.3)
- added D17: Red, LED_SMD:LED_0805_2012Metric, F.Cu at (151.8, -7.21)
- added D23: Red, LED_SMD:LED_0805_2012Metric, F.Cu at (151.8, -4.17)
- added D24: Red, LED_SMD:LED_0805_2012Metric, F.Cu at (151.8, -1.14)
- added D25: BZT52C16, Diode_SMD:D_SOD-123, F.Cu at (170.2, -6.13)
- added JP4: Jumper_3_Open, Connector_PinHeader_2.54mm:PinHeader_1x03_P2.54mm_Vertical, F.Cu at (140.2, -33.1)
- added Q10: SI2347DS-T1-GE3, Package_TO_SOT_SMD:SOT-23-3, F.Cu at (147.0, -19.1)
- added Q11: MMBT3904L RFG, Package_TO_SOT_SMD:SOT-23-3, F.Cu at (147.0, -14.5)
- added Q15: SI2318CDS-T1-GE3, Package_TO_SOT_SMD:SOT-23-3, F.Cu at (147.0, -9.90)
- added Q7: SI2318CDS-T1-GE3, Package_TO_SOT_SMD:SOT-23-3, F.Cu at (147.0, -33.0)
- added Q8: SI2347DS-T1-GE3, Package_TO_SOT_SMD:SOT-23-3, F.Cu at (147.0, -28.4)
- added Q9: MMBT3904L RFG, Package_TO_SOT_SMD:SOT-23-3, F.Cu at (147.0, -23.8)
- added R100: 120k, Resistor_SMD:R_0603_1608Metric_Pad0.98x0.95mm_HandSolder, F.Cu at (164.8, -24.1)
- added R101: 100k, Resistor_SMD:R_0603_1608Metric_Pad0.98x0.95mm_HandSolder, F.Cu at (164.8, -21.6)
- added R102: 3k, Resistor_SMD:R_0603_1608Metric_Pad0.98x0.95mm_HandSolder, F.Cu at (164.8, -19.1)
- added R103: 510, Resistor_SMD:R_0603_1608Metric_Pad0.98x0.95mm_HandSolder, F.Cu at (169.2, -34.2)
- added R104: 510, Resistor_SMD:R_0603_1608Metric_Pad0.98x0.95mm_HandSolder, F.Cu at (169.2, -31.7)
- added R105: 100k, Resistor_SMD:R_0603_1608Metric_Pad0.98x0.95mm_HandSolder, F.Cu at (169.2, -29.1)
- added R106: 100k, Resistor_SMD:R_0603_1608Metric_Pad0.98x0.95mm_HandSolder, F.Cu at (169.2, -26.6)
- added R107: 100k, Resistor_SMD:R_0603_1608Metric_Pad0.98x0.95mm_HandSolder, F.Cu at (169.2, -24.1)
- added R108: 510, Resistor_SMD:R_0603_1608Metric_Pad0.98x0.95mm_HandSolder, F.Cu at (169.2, -21.6)
- added R109: 510, Resistor_SMD:R_0603_1608Metric_Pad0.98x0.95mm_HandSolder, F.Cu at (169.2, -19.1)
- added R40: 100, Resistor_SMD:R_0603_1608Metric_Pad0.98x0.95mm_HandSolder, F.Cu at (151.8, -24.1)
- added R57: 100k, Resistor_SMD:R_0603_1608Metric_Pad0.98x0.95mm_HandSolder, F.Cu at (151.8, -21.6)
- added R65: 10k, Resistor_SMD:R_0603_1608Metric_Pad0.98x0.95mm_HandSolder, F.Cu at (151.8, -19.1)
- added R71: 100k, Resistor_SMD:R_0603_1608Metric_Pad0.98x0.95mm_HandSolder, F.Cu at (156.1, -34.2)
- added R79: 510, Resistor_SMD:R_0603_1608Metric_Pad0.98x0.95mm_HandSolder, F.Cu at (156.1, -31.7)
- added R80: 0, Resistor_SMD:R_0603_1608Metric_Pad0.98x0.95mm_HandSolder, F.Cu at (156.1, -29.1)
- added R81: 0, Resistor_SMD:R_0603_1608Metric_Pad0.98x0.95mm_HandSolder, F.Cu at (156.1, -26.6)
- added R82: 0, Resistor_SMD:R_0603_1608Metric_Pad0.98x0.95mm_HandSolder, F.Cu at (156.1, -24.1)
- added R83: 51, Resistor_SMD:R_0603_1608Metric_Pad0.98x0.95mm_HandSolder, F.Cu at (156.1, -21.6)
- added R84: 0, Resistor_SMD:R_0603_1608Metric_Pad0.98x0.95mm_HandSolder, F.Cu at (156.1, -19.1)
- added R85: 510, Resistor_SMD:R_0603_1608Metric_Pad0.98x0.95mm_HandSolder, F.Cu at (160.5, -34.2)
- added R86: 10k, Resistor_SMD:R_0603_1608Metric_Pad0.98x0.95mm_HandSolder, F.Cu at (160.5, -31.7)
- added R87: 100k, Resistor_SMD:R_0603_1608Metric_Pad0.98x0.95mm_HandSolder, F.Cu at (160.5, -29.1)
- added R88: 100k, Resistor_SMD:R_0603_1608Metric_Pad0.98x0.95mm_HandSolder, F.Cu at (160.5, -26.6)
- added R89: 120, Resistor_SMD:R_0603_1608Metric_Pad0.98x0.95mm_HandSolder, F.Cu at (140.0, -24.5)
- added R90: 100k, Resistor_SMD:R_0603_1608Metric_Pad0.98x0.95mm_HandSolder, F.Cu at (160.5, -24.1)
- added R92: 1k, Resistor_SMD:R_0603_1608Metric_Pad0.98x0.95mm_HandSolder, F.Cu at (160.5, -21.6)
- added R94: 10k, Resistor_SMD:R_0603_1608Metric_Pad0.98x0.95mm_HandSolder, F.Cu at (160.5, -19.1)
- added R96: 10k, Resistor_SMD:R_0603_1608Metric_Pad0.98x0.95mm_HandSolder, F.Cu at (164.8, -34.2)
- added R97: 10k, Resistor_SMD:R_0603_1608Metric_Pad0.98x0.95mm_HandSolder, F.Cu at (164.8, -31.7)
- added R98: 3M, Resistor_SMD:R_0603_1608Metric_Pad0.98x0.95mm_HandSolder, F.Cu at (164.8, -29.1)
- added R99: 30k, Resistor_SMD:R_0603_1608Metric_Pad0.98x0.95mm_HandSolder, F.Cu at (164.8, -26.6)
- added RV2: 100k, Potentiometer_SMD:Potentiometer_Bourns_TC33X_Vertical, F.Cu at (157.2, -15.5)
- added RV5: 100k, Potentiometer_SMD:Potentiometer_Bourns_TC33X_Vertical, F.Cu at (157.2, -10.7)
- added RV6: 100k, Potentiometer_SMD:Potentiometer_Bourns_TC33X_Vertical, F.Cu at (157.2, -5.98)
- added TP60: ~, TestPoint:TestPoint_Pad_1.5x1.5mm, F.Cu at (162.0, -16.1)
- added TP63: ~, TestPoint:TestPoint_Pad_1.5x1.5mm, F.Cu at (162.0, -12.5)
- added TP64: ~, TestPoint:TestPoint_Pad_1.5x1.5mm, F.Cu at (162.0, -8.98)
- added TP65: ~, TestPoint:TestPoint_Pad_1.5x1.5mm, F.Cu at (162.0, -5.43)
- added TP67: ~, TestPoint:TestPoint_Pad_1.5x1.5mm, F.Cu at (165.5, -16.1)
- added TP68: ~, TestPoint:TestPoint_Pad_1.5x1.5mm, F.Cu at (165.5, -12.5)
- added TP69: ~, TestPoint:TestPoint_Pad_1.5x1.5mm, F.Cu at (165.5, -8.98)
- added U15: LM393BIDR, Package_SO:SOIC-8_3.9x4.9mm_P1.27mm, F.Cu at (177.3, -14.5)
- added U16: LM393BIDR, Package_SO:SOIC-8_3.9x4.9mm_P1.27mm, F.Cu at (177.3, -7.92)
- added U17: ~, 20pinMX150Header:CONN_SD-19427-025_MOL, F.Cu at (88.7, 43.6)
- added U18: ~, 20pinMX150Header:CONN_SD-19427-025_MOL, F.Cu at (175.1, 43.6)
- added U19: ~, 20pinMX150Header:CONN_SD-19427-025_MOL, F.Cu at (261.4, 43.6)
- added U4: CD4002BM96, Package_SO:SOIC-14_3.9x8.7mm_P1.27mm, F.Cu at (175.6, -30.2)
- R32: moved to B.Cu
- moved R3 88.3 mm to (318.6, 81.4)
- moved D4 88.3 mm to (322.6, 86.3)
- moved D7 88.3 mm to (322.5, 81.4)
- moved R1 88.3 mm to (318.8, 86.2)
- moved TP49 88.3 mm to (322.6, 73.3)
- moved TP56 88.3 mm to (322.6, 54.3)
- moved TP57 88.3 mm to (322.6, 59.1)
- moved TP58 88.3 mm to (322.6, 63.8)
- moved TP59 88.3 mm to (322.6, 68.6)
- moved C10 83.6 mm to (227.4, 77.0)
- moved C11 83.6 mm to (219.1, 91.0)
- moved C8 83.6 mm to (226.6, 73.2)
- moved D2 83.6 mm to (232.7, 77.0)
- moved D5 83.6 mm to (251.5, 87.6)
- moved D6 83.6 mm to (253.5, 94.6)
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Connections:
- net /Connector-Root/BSE-SIG renamed /BSE-SIG
- net /Connector-Root/BSPD-FAULT renamed /BSPD-FAULT
Routing:
- net +12V: track 65.3 -> 778.7 mm, vias 26 -> 0
- net /BRUHbus/CAN2_H: track 295.9 -> 0.00 mm, vias 2 -> 0
- net /BRUHbus/CAN2_L: track 302.4 -> 27.5 mm, vias 3 -> 0
- net /STM32-Root/STM32H723ZGT6/PA0: track 270.1 -> 0.00 mm, vias 1 -> 0
- net /STM32-Root/STM32H723ZGT6/PA1: track 268.3 -> 0.00 mm, vias 1 -> 0
- net /STM32-Root/STM32H723ZGT6/PA2: track 262.6 -> 0.00 mm, vias 1 -> 0
- net /STM32-Root/STM32H723ZGT6/PB12: track 215.6 -> 0.00 mm, vias 2 -> 0
- net GND: track 237.2 -> 441.4 mm, vias 191 -> 0
- net /STM32-Root/STM32H723ZGT6/PG11: track 194.1 -> 0.00 mm, vias 1 -> 0
- net /STM32-Root/STM32H723ZGT6/PF8: track 191.4 -> 0.00 mm, vias 1 -> 0
- net /STM32-Root/STM32H723ZGT6/PG6: track 190.4 -> 0.00 mm, vias 1 -> 0
- net /STM32-Root/STM32H723ZGT6/PG12: track 190.3 -> 0.00 mm, vias 1 -> 0
- net /STM32-Root/STM32H723ZGT6/PG7: track 189.5 -> 0.00 mm, vias 1 -> 0
- net /STM32-Root/STM32H723ZGT6/PG8: track 188.4 -> 0.00 mm, vias 1 -> 0
- net /STM32-Root/STM32H723ZGT6/PC2: track 187.1 -> 0.00 mm, vias 1 -> 0
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- removed copper zone on F.Cu, net +12V
- removed copper zone on In2.Cu, net +12V
- removed copper zone on F.Cu, net +3.3V
- removed copper zone on In2.Cu, net +3.3V
- removed copper zone on F.Cu, net +4.8V
- removed copper zone on F.Cu, net +5V
- removed copper zone on In2.Cu, net +5V
- removed copper zone on F.Cu, net /Connector-Root/SPEAKER+
- removed copper zone on F.Cu, net /Connector-Root/SPEAKER-
- removed copper zone on F.Cu, net /Connector-Root/Vin+
- removed copper zone on F.Cu, net GND
- removed copper zone on In1.Cu, net GND
- removed copper zone on F.Cu, net Net-(D2-K)
Other:
- board outline removed

Commit message: going bald
Routing:
- net +12V: track 778.7 -> 0.00 mm
- net GND: track 441.4 -> 0.00 mm
- net /STM32-Root/STM32H723ZGT6/PG15: track 194.4 -> 0.00 mm
- net /STM32-Root/STM32H723ZGT6/PG13: track 190.5 -> 0.00 mm
- net /STM32-Root/STM32H723ZGT6/PG10: track 189.8 -> 0.00 mm
- net /STM32-Root/STM32H723ZGT6/PG14: track 188.6 -> 0.00 mm
- net /STM32-Root/STM32H723ZGT6/PG9: track 182.1 -> 0.00 mm
- net +3.3V: track 172.2 -> 0.00 mm
- net /STM32-Root/STM32H723ZGT6/PE11: track 169.8 -> 0.00 mm
- net /STM32-Root/STM32H723ZGT6/PE10: track 167.9 -> 0.00 mm
- net /STM32-Root/STM32H723ZGT6/PB5: track 166.6 -> 0.00 mm
- net /BSPD-FAULT: track 136.2 -> 0.00 mm
- net /Connector-Root/IMD-FAULT: track 121.7 -> 0.00 mm
- net /Connector-Root/BMS-FAULT: track 120.0 -> 0.00 mm
- net /BRUHbus/CAN1_L: track 111.0 -> 0.00 mm
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- removed copper zone on B.Cu, net /Connector-Root/Vin+

Commit message: slimed ethernet
Parts:
- removed J6, J7, J8: BRUHBus, Connector_RJ:RJ45_Amphenol_RJHSE538X
- removed Q2, Q6: BSD235NH6327XT, Package_TO_SOT_SMD:SOT-363_SC-70-6_Handsoldering
- removed R12, R17, R18, R21, R38, R39: 2.4k, Resistor_SMD:R_0603_1608Metric_Pad0.98x0.95mm_HandSolder
- removed R33, R35, R37: 0, Resistor_SMD:R_0805_2012Metric_Pad1.20x1.40mm_HandSolder
- removed R34, R75, R76: 10k, Resistor_SMD:R_0603_1608Metric_Pad0.98x0.95mm_HandSolder
- removed R36, R77, R78: 100, Resistor_SMD:R_0603_1608Metric_Pad0.98x0.95mm_HandSolder
- R32: moved to F.Cu
- moved R102 145.5 mm to (206.9, 120.2)
- moved R96 145.5 mm to (206.9, 105.1)
- moved R97 145.5 mm to (206.9, 107.6)
- moved C42 145.5 mm to (193.9, 107.6)
- moved C86 145.5 mm to (193.9, 112.6)
- moved D12 145.5 mm to (212.3, 126.5)
- moved D13 145.5 mm to (194.0, 123.0)
- moved D17 145.5 mm to (194.0, 132.1)
- moved D23 145.5 mm to (194.0, 135.1)
- moved Q15 145.5 mm to (189.1, 129.4)
- moved R101 145.5 mm to (206.9, 117.7)
- moved R103 145.5 mm to (211.3, 105.1)
- moved R104 145.5 mm to (211.3, 107.6)
- moved R106 145.5 mm to (211.3, 112.6)
- moved R107 145.5 mm to (211.3, 115.2)
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Connections:
- net /BRUHbus/CAN1_H renamed /Connector-Root/CAN1_H
- net /BRUHbus/CAN1_L renamed /Connector-Root/CAN1_L
- JP3 pad 3: /BRUHbus/CAN2_L -> /Connector-Root/CAN2_L
- R42 pad 1: /BRUHbus/CAN2_H -> /Connector-Root/CAN2_H
- TP22 pad 1: /BRUHbus/CAN2_H -> /Connector-Root/CAN2_H
- TP23 pad 1: /BRUHbus/CAN2_L -> /Connector-Root/CAN2_L
- U12 pad 6: /BRUHbus/CAN2_L -> /Connector-Root/CAN2_L
- U12 pad 7: /BRUHbus/CAN2_H -> /Connector-Root/CAN2_H
- U18 pad 10: /STM32-Root/STM32H723ZGT6/PG11 -> /Connector-Root/CAN2_L
- U18 pad 11: /STM32-Root/STM32H723ZGT6/PG10 -> /Connector-Root/CAN2_H
- U18 pad 3: /Connector-Root/Isense-active -> /BSPD-Logic/Isense-active

Commit message: placements lowkenuinely done
Parts:
- removed R92: 1k, Resistor_SMD:R_0603_1608Metric_Pad0.98x0.95mm_HandSolder
- added R12: 0, Resistor_SMD:R_0603_1608Metric_Pad0.98x0.95mm_HandSolder, F.Cu at (114.0, 84.1)
- moved U16 118.5 mm to (109.1, 88.1), turned to 180 degrees
- moved TP64 107.3 mm to (107.5, 83.7)
- moved RV6 106.9 mm to (102.2, 88.8)
- moved RV5 106.6 mm to (102.2, 84.6)
- moved R87 105.2 mm to (101.3, 81.6)
- moved D12 104.5 mm to (112.2, 96.8), turned to 180 degrees
- moved R88 103.5 mm to (101.3, 91.7), turned to 180 degrees
- moved TP63 102.3 mm to (111.3, 83.7)
- moved R108 100.8 mm to (111.4, 104.2), turned to 90 degrees
- moved R109 98.9 mm to (113.7, 104.2), turned to 90 degrees
- moved R97 95.9 mm to (112.1, 93.4), turned to -90 degrees
- moved D15 94.1 mm to (122.5, 102.1)
- moved R105 94.0 mm to (117.6, 102.0), turned to 90 degrees
- moved R90 93.9 mm to (115.0, 81.4), turned to 180 degrees
- moved R96 93.6 mm to (114.1, 93.4), turned to -90 degrees
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