File: VCU_v2/bspd.kicad_sch (KiCad schematic)
At the start: 0 parts

Commit message: bspd schematic done
Parts:
- added C41, C42, C44, C86: 100nF, Capacitor_SMD:C_0603_1608Metric_Pad1.08x0.95mm_HandSolder, symbol -C-Ceramic-0603:C-0603-100nF-10%-50V-X7R
- added D1, D12, D15, D25: BZT52C16, Diode_SMD:D_SOD-123, symbol -Diodes-Zener:BZT52C16
- added D13, D14, D16, D17, D23, D24: Red, LED_SMD:LED_0805_2012Metric, symbol -Diodes-LED:NCD0805R1
- added Q10, Q8: SI2347DS-T1-GE3, Package_TO_SOT_SMD:SOT-23-3, symbol -MOSFET-P-Channel:SI2347DS-T1-GE3
- added Q11, Q9: MMBT3904L RFG, Package_TO_SOT_SMD:SOT-23-3, symbol -BJT-NPN:MMBT3904L-RFG
- added Q15, Q7: SI2318CDS-T1-GE3, Package_TO_SOT_SMD:SOT-23-3, symbol -MOSFET-N-Channel:SI2318CDS-T1-GE3
- added R100: 120k, Resistor_SMD:R_0603_1608Metric_Pad0.98x0.95mm_HandSolder, symbol -R-SMD-0603:R-0603-120k-1%-100mW-100PPM
- added R101, R105, R106, R107, R57, R71, R87, R88, R90: 100k, Resistor_SMD:R_0603_1608Metric_Pad0.98x0.95mm_HandSolder, symbol -R-SMD-0603:R-0603-100k-1%-100mW-100PPM
- added R102: 3k, Resistor_SMD:R_0603_1608Metric_Pad0.98x0.95mm_HandSolder, symbol -R-SMD-0603:R-0603-3k-1%-100mW-100PPM
- added R103, R104, R108, R109, R79, R85: 510, Resistor_SMD:R_0603_1608Metric_Pad0.98x0.95mm_HandSolder, symbol -R-SMD-0603:R-0603-510-1%-100mW-100PPM
- added R40: 100, Resistor_SMD:R_0603_1608Metric_Pad0.98x0.95mm_HandSolder, symbol BFR Resistors:RMCF0603FT100R
- added R65, R86: 10k, Resistor_SMD:R_0603_1608Metric_Pad0.98x0.95mm_HandSolder, symbol BFR Resistors:RMCF0603FT10K0
- added R80, R81, R82, R84: 0, Resistor_SMD:R_0603_1608Metric_Pad0.98x0.95mm_HandSolder, symbol -R-SMD-0603:R-0603-0-1%-100mW-1500PPM
- added R83: 51, Resistor_SMD:R_0603_1608Metric_Pad0.98x0.95mm_HandSolder, symbol -R-SMD-0603:R-0603-51-1%-100mW-100PPM
- added R92: 1k, Resistor_SMD:R_0603_1608Metric_Pad0.98x0.95mm_HandSolder, symbol -R-SMD-0603:R-0603-1k-1%-100mW-100PPM
- added R94, R96, R97: 10k, Resistor_SMD:R_0603_1608Metric_Pad0.98x0.95mm_HandSolder, symbol -R-SMD-0603:R-0603-10k-1%-100mW-100PPM
- added R98: 3M, Resistor_SMD:R_0603_1608Metric_Pad0.98x0.95mm_HandSolder, symbol -R-SMD-0603:R-0603-3M-1%-100mW-100PPM
- added R99: 30k, Resistor_SMD:R_0603_1608Metric_Pad0.98x0.95mm_HandSolder, symbol -R-SMD-0603:R-0603-30k-1%-100mW-100PPM
- added RV2, RV5, RV6: 100k, Potentiometer_SMD:Potentiometer_Bourns_TC33X_Vertical, symbol -Potentiometers:TC33X-2-104E
- added TP60, TP63, TP64, TP65, TP67, TP68, TP69: ~, TestPoint:TestPoint_Pad_1.5x1.5mm, symbol -Test-Points:Square-Pad-1.5mm
- added U15, U16: LM393BIDR, Package_SO:SOIC-8_3.9x4.9mm_P1.27mm, symbol -Comparators:LM393BIDR
- added U4: CD4002BM96, Package_SO:SOIC-14_3.9x8.7mm_P1.27mm, symbol -Logic-Gates:CD4002BM96
Connections:
- net Isense-active: now also U4.4, U4.5
- net Isense-thresh: now also U4.10, U4.9
- new net: D1.1 (K), Q7.1 (G), R40.2
- new net: Q11.1 (B), R107.2
- new net: Q11.3 (C), Q9.2 (E)
- new net: R98.1, U4.1
- new net: C41.2, R98.2, U15.2 (-)
- new net: D15.2 (A), Q10.1 (G), R101.2
- new net: RV6.2, TP64.1, U16.6 (-)
- new net: Q9.1 (B), R106.2
- new net: R96.1, U16.1, U4.11
- new net: R92.2, U16.2 (-), U16.5 (+)
- new net: RV5.2, TP63.1, U16.3 (+)
- new net: R81.1, R82.2, R84.1
- new net: D23.2 (A), R79.1
- new net: R80.2, R84.2, TP60.1, U15.5 (+)
- new net: R87.1, RV5.1
- new net: Q10.3 (D), R103.2, R104.2
- new net: R88.2, RV6.3
- new net: R101.1, R107.1, TP67.1, U4.13
- new net: R102.1, R105.1, R106.1, TP68.1, U15.1
- new net: R100.2, R99.1, U15.3 (+)
- new net: D14.2 (A), R109.1
- new net: Q8.3 (D), R108.2, R109.2
- new net: R97.1, U16.7, U4.12
- new net: D23.1 (K), D24.1 (K), Q15.3 (D)
- new net: D24.2 (A), R85.1
- new net: D25.2 (A), Q15.2 (S), R83.2
- new net: R94.1, TP65.1, U15.7, U4.2, U4.3
- new net: D12.2 (A), Q8.1 (G), R105.2
- new net: D16.2 (A), R103.1
- new net: D17.2 (A), R104.1
- new net: D13.2 (A), R108.1
- new net: R57.1, RV2.1
- new net: R80.1, RV2.2
- new net +12V: R65.1, R79.2, R85.2, R86.2
- new net 12V: C42.2, C44.2, C86.2, D12.1 (K), D15.1 (K), Q10.2 (S), Q8.2 (S), R102.2, R57.2, R81.2, R87.2, R94.2, R96.2, R97.2, R99.2, RV6.1, U15.8 (VCC), U16.8 (VCC), U4.14 (VDD)
- new net BSE: R90.2, R92.1, U15.6 (-)
- new net BSPD-OUT: Q7.3 (D), R65.2
- new net BSPD-inv: D25.1 (K), Q15.1 (G), Q9.3 (C), R40.1, R71.1, R71.2, R86.1, TP69.1
- new net GND: C41.1, C42.1, C44.1, C86.1, D1.2 (A), D13.1 (K), D14.1 (K), D16.1 (K), D17.1 (K), Q11.2 (E), Q7.2 (S), R100.1, R82.1, R83.1, R88.1, R90.1, RV2.3, RV5.3, U15.4 (GND), U16.4 (GND), U4.7 (VSS)
- no-connect marks 0 -> 2
Other:
- note added: "BSPD-Logic"
- note added: "BSPD_INV"
- note added: "Bound check for BRK (LOW=BRAKING)"
- note added: "Bound check for CURR (LOW=MUCH CURRENT)"
- note added: "Brake High thresh"
- note added: "Brake Low Thresh"
- note added: "Brake Plausibility"
- note added: "Brake Thresh"
- note added: "Delayed Plausibility Check (LOW=FAULT)"
- note added: "LOW = BRK_PRES1_OUT passed short-to-12V test"
- note added: "LOW = BRK_PRES1_OUT passed short-to-GND test"
- note added: "LOW = some signal is invalid"
- note added: "Signal Validity"

Commit message: vcu v2 schematics done
Parts:
- renumbered C41 to C81, C42 to C82, C44 to C83, C86 to C84, D12 to D10, D13 to D11, D14 to D12, D1 to D13, D23 to D14, D25 to D15, D24 to D16, D15 to D7, D16 to D8, D17 to D9, Q8 to Q10, Q7 to Q11, Q15 to Q12, Q10 to Q7, Q9 to Q8, Q11 to Q9, R109 to R100, R40 to R101, R71 to R102, R79 to R103, R83 to R104, R85 to R105, R57 to R75, R87 to R76, R88 to R77, R80 to R78, R81 to R79, R82 to R80, R90 to R81, R84 to R82, R92 to R83, R96 to R84, R97 to R85, R94 to R86, R98 to R87, R99 to R88, R100 to R89, R101 to R90, R103 to R91, R104 to R92, R102 to R93, R106 to R94, R107 to R95, R86 to R96, R105 to R97, R108 to R98, R65 to R99, RV2 to RV1, RV5 to RV2, RV6 to RV3, TP63 to TP59, TP64 to TP60, TP60 to TP61, TP65 to TP62, TP67 to TP63, TP69 to TP64, TP68 to TP65, U16 to U14, U4 to U16

Commit message: placements friggin 80% friggin done shoutout epstein
Parts:
- renumbered C81 to C41, C82 to C42, C83 to C44, C84 to C86, D13 to D1, D10 to D12, D11 to D13, D12 to D14, D7 to D15, D8 to D16, D9 to D17, D14 to D23, D16 to D24, D15 to D25, Q7 to Q10, Q9 to Q11, Q12 to Q15, Q11 to Q7, Q10 to Q8, Q8 to Q9, R89 to R100, R90 to R101, R93 to R102, R91 to R103, R92 to R104, R97 to R105, R94 to R106, R95 to R107, R98 to R108, R100 to R109, R101 to R40, R75 to R57, R99 to R65, R102 to R71, R103 to R79, R78 to R80, R79 to R81, R80 to R82, R104 to R83, R82 to R84, R105 to R85, R96 to R86, R76 to R87, R77 to R88, R81 to R90, R83 to R92, R86 to R94, R84 to R96, R85 to R97, R87 to R98, R88 to R99, RV1 to RV2, RV2 to RV5, RV3 to RV6, TP61 to TP60, TP59 to TP63, TP60 to TP64, TP62 to TP65, TP63 to TP67, TP65 to TP68, TP64 to TP69, U14 to U16, U16 to U4
Connections:
- net BSPD-inv: no longer D25.1 (K), Q15.1 (G), R71.2
- new net: D25.1 (K), Q15.1 (G), R71.2

Commit message: added hella comments to bspd logic
Parts:
- removed R92: 1k, Resistor_SMD:R_0603_1608Metric_Pad0.98x0.95mm_HandSolder, symbol -R-SMD-0603:R-0603-1k-1%-100mW-100PPM
- added R12: 0, Resistor_SMD:R_0603_1608Metric_Pad0.98x0.95mm_HandSolder, symbol -R-SMD-0603:R-0603-0-1%-100mW-1500PPM
Connections:
- net BSE: now also R12.1
- net at U16.2 (-), U16.5 (+): now also R12.2

Commit message: vcu v2 done
Connections:
- net +12V: now also C44.2, C86.2, D12.1 (K), D15.1 (K), Q10.2 (S), Q8.2 (S), R102.2, R57.2, R81.2, R87.2, R94.2, R96.2, R97.2, R99.2, RV6.1, U16.8 (VCC), U4.14 (VDD)
- removed net 12V: C42.2, C44.2, C86.2, D12.1 (K), D15.1 (K), Q10.2 (S), Q8.2 (S), R102.2, R57.2, R81.2, R87.2, R94.2, R96.2, R97.2, R99.2, RV6.1, U15.8 (VCC), U16.8 (VCC), U4.14 (VDD)
- new net: C42.2, U15.8 (VCC)
